File: hw/Esp8266AquariumLight.kicad_pcb (KiCad board)
At the start: 2 copper layers, 99.9 x 29 mm, 34 parts, among them J1 POWER, J2 Conn_02x03_Odd_Even, J3 Conn_01x03, J4 Conn_01x04, Q1 S8050, Q2 S8050, Q3 AO3401A, SW2 RST, SW3 PGM, U1 AMS1117-3.3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

Commit message: update: assembly pictures
Parts:
- added REF**: KiCad-Logo2_5mm_SilkScreen, Symbol:KiCad-Logo2_5mm_SilkScreen, B.Cu at (112.3, 109.5)
- added REF**: OSHW-Logo2_7.3x6mm_SilkScreen, Symbol:OSHW-Logo2_7.3x6mm_SilkScreen, B.Cu at (126.2, 110.0)
Other:
- board text added: "https://github.com/gvoigtlaender/Esp8266AquariumLight"
- board text removed: "gvoigtlaender@googlemail.com"
